Commit message: Update

File: robosys_description/urdf/robosys.urdf (robot description, URDF)
Before this commit: robot robosys, 3 links, 2 joints
Links:
- added link depth_base_link
- added link depth_link, mass 0.1; collision box size=0.01 0.01 0.01; visual box size=0.01 0.01 0.01
Joints:
- added joint depth_base_joint: type fixed, parent base_link, child depth_base_link, origin xyz=0.095 0 0.05 rpy=0 0 0
- added joint depth_joint: type fixed, parent depth_base_link, child depth_link, origin xyz=0 0 0.005 rpy=0 0 0

Commit message: update

File: robosys_description/urdf/robosys.urdf (robot description, URDF)
Before this commit: robot robosys, 5 links, 4 joints
Links:
- removed link depth_base_link
Joints:
- removed joint depth_joint
- joint depth_base_joint: child depth_base_link -> depth_link; origin xyz=0.095 0 0.05 rpy=0 0 0 -> xyz=0.1 0 0.055 rpy=0 0 0

Commit message: Add Depth_Camera

File: robosys_description/urdf/robosys.urdf (robot description, URDF)
Before this commit: robot robosys, 4 links, 3 joints
Links:
- added link body, mass 1.0; collision box size=0.2 0.1 0.1; visual box size=0.2 0.1 0.1
- link base_link: mass 1.0 -> None; geometry 
Joints:
- added joint world_joint: type fixed, parent base_link, child body, origin xyz=0 0 0 rpy=0 0 0
- joint depth_base_joint: parent base_link -> body
- joint left_j: parent base_link -> body
- joint right_j: parent base_link -> body

Commit message: Add center_wheel

File: robosys_description/urdf/robosys.urdf (robot description, URDF)
Before this commit: robot robosys, 5 links, 4 joints
Links:
- added link center_link, mass 1.0; collision box size=0.05 0.025 0.025; visual box size=0.05 0.025 0.025
- added link center_wheel, mass 0.5; collision cylinder length=0.04 radius=0.0175; visual cylinder length=0.04 radius=0.0175
Joints:
- added joint center_link_j: type continuous, parent body, child center_link, origin xyz=0.095 0 -0.05 rpy=0 0 0, axis 0 0 1
- added joint center_wheel_j: type continuous, parent center_link, child center_wheel, origin xyz=-0.04 0 -0.0125 rpy=0 0 0, axis 0 1 0
- joint depth_base_joint: axis (none) -> 0 1 0
- joint world_joint: origin xyz=0 0 0 rpy=0 0 0 -> xyz=0 0 1 rpy=0 0 0
